Commit message: updating ES with saving

File: opendog.urdf (robot description, URDF)
Before this commit: robot test_robot, 13 links, 12 joints
Joints:
- joint joint1: limit (none) -> lower=-1.0 upper=1.0 effort=300 velocity=12; type continuous -> revolute
- joint joint10: limit (none) -> lower=-1.0 upper=1.0 effort=300 velocity=12; type continuous -> revolute
- joint joint11: limit (none) -> lower=-1.0 upper=1.0 effort=300 velocity=12; type continuous -> revolute
- joint joint12: limit (none) -> lower=-1.0 upper=1.0 effort=300 velocity=12; type continuous -> revolute
- joint joint2: limit (none) -> lower=-1.0 upper=1.0 effort=300 velocity=12; type continuous -> revolute
- joint joint3: limit (none) -> lower=-1.0 upper=1.0 effort=300 velocity=12; type continuous -> revolute
- joint joint4: limit (none) -> lower=-1.0 upper=1.0 effort=300 velocity=12; type continuous -> revolute
- joint joint5: limit (none) -> lower=-1.0 upper=1.0 effort=300 velocity=12; type continuous -> revolute
- joint joint6: limit (none) -> lower=-1.0 upper=1.0 effort=300 velocity=12; type continuous -> revolute
- joint joint7: limit (none) -> lower=-1.0 upper=1.0 effort=300 velocity=12; type continuous -> revolute
- joint joint8: limit (none) -> lower=-1.0 upper=1.0 effort=300 velocity=12; type continuous -> revolute
- joint joint9: limit (none) -> lower=-1.0 upper=1.0 effort=300 velocity=12; type continuous -> revolute

Commit message: OpenDog First Steps

File: opendog.urdf (robot description, URDF)
Before this commit: robot test_robot, 13 links, 12 joints
Joints:
- joint joint1: limit lower=-1.0 upper=1.0 effort=300 velocity=12 -> lower=-1.0 upper=1.0 effort=500 velocity=12
- joint joint10: limit lower=-1.0 upper=1.0 effort=300 velocity=12 -> lower=-1.0 upper=1.0 effort=500 velocity=12
- joint joint11: limit lower=-1.0 upper=1.0 effort=300 velocity=12 -> lower=-1.0 upper=1.0 effort=500 velocity=12
- joint joint12: limit lower=-1.0 upper=1.0 effort=300 velocity=12 -> lower=-1.0 upper=1.0 effort=500 velocity=12
- joint joint2: limit lower=-1.0 upper=1.0 effort=300 velocity=12 -> lower=-1.0 upper=1.0 effort=500 velocity=12
- joint joint3: limit lower=-1.0 upper=1.0 effort=300 velocity=12 -> lower=-1.0 upper=1.0 effort=500 velocity=12
- joint joint4: limit lower=-1.0 upper=1.0 effort=300 velocity=12 -> lower=-1.0 upper=1.0 effort=500 velocity=12
- joint joint5: limit lower=-1.0 upper=1.0 effort=300 velocity=12 -> lower=-1.0 upper=1.0 effort=500 velocity=12
- joint joint6: limit lower=-1.0 upper=1.0 effort=300 velocity=12 -> lower=-1.0 upper=1.0 effort=500 velocity=12
- joint joint7: limit lower=-1.0 upper=1.0 effort=300 velocity=12 -> lower=-1.0 upper=1.0 effort=500 velocity=12
- joint joint8: limit lower=-1.0 upper=1.0 effort=300 velocity=12 -> lower=-1.0 upper=1.0 effort=500 velocity=12
- joint joint9: limit lower=-1.0 upper=1.0 effort=300 velocity=12 -> lower=-1.0 upper=1.0 effort=500 velocity=12
